File: hardware/usb_uart.sch (KiCad schematic (older format))
At the start: 12 parts

Commit message: Added hierarchical connections and labels clean up.
Signed-off-by: Kamil Gardziejczyk <kamil.gardziejczyk@firmwave.com>
Parts:
- added D? (x2): LED, symbol LED
- added R? (x2): 220, symbol R
- R? (x2): value R -> 0
Connections:
- net labels added: CTS, DCD, DSR, DTR, GPIO.2, GPIO.3, GPIO.4, GPIO.5, GPIO.6, RI, RTS, RXD, TXD
- wire segments 49 -> 78
Other:
- moved on the sheet: D?, FL?, J?, L?, R?

Commit message: Adding missing connections for battery charger IC.
Signed-off-by: Kamil Gardziejczyk <kamil.gardziejczyk@firmwave.com>
Connections:
- net labels added: USB_CHR0, USB_CHR1, USB_CHREN
- net labels removed: VBUS
- wire segments 78 -> 81
Changed lines of the file:
@@
 L GND #PWR?
 U 1 1 597CACA2
-P 1400 4450
-F 0 "#PWR?" H 1400 4200 50  0001 C CNN
-F 1 "GND" H 1400 4300 50  0000 C CNN
-F 2 "" H 1400 4450 50  0001 C CNN
-F 3 "" H 1400 4450 50  0001 C CNN
-	1    1400 4450
+P 1550 4450
+F 0 "#PWR?" H 1550 4200 50  0001 C CNN
+F 1 "GND" H 1550 4300 50  0000 C CNN
+F 2 "" H 1550 4450 50  0001 C CNN
+F 3 "" H 1550 4450 50  0001 C CNN
+	1    1550 4450
 	1    0    0    -1
 $EndComp
@@
 	1    0    0    -1
 $EndComp
-$Comp
-L PWR_FLAG #FLG?
-U 1 1 597CB023
-P 2100 3050
-F 0 "#FLG?" H 2100 3125 50  0001 C CNN
-F 1 "PWR_FLAG" H 2100 3200 50  0000 C CNN
-F 2 "" H 2100 3050 50  0001 C CNN
-F 3 "" H 2100 3050 50  0001 C CNN
-	1    2100 3050
-	1    0    0    -1
-$EndComp
-Text GLabel 2050 3100 0    60   Input ~ 0
-VUSB
-Text GLabel 4200 4100 0    60   Input ~ 0
-VUSB
 $Comp
 L GND #PWR?
@@
 Text Label 2750 4900 0    60   ~ 0
 D-
-Text GLabel 1750 4700 0    60   Input ~ 0
-VBUS
 $Comp
 L GND #PWR?
@@
 	1    0    0    -1
 $EndComp
-Text GLabel 5450 4850 3    60   Input ~ 0
-VBUS
 $Comp
 L VDD #PWR?
@@
 	2100 3050 2100 3200
 Wire Wire Line
-	2100 3100 2050 3100
-Connection ~ 2100 3100
-Wire Wire Line
 	4600 3700 4850 3700
 Wire Wire Line
@@
 Wire Wire Line
 	3850 2600 4150 2600
-Wire Wire Line
-	1750 4700 1900 4700
 Wire Wire Line
 	5450 4850 5450 4700
@@
 Wire Wire Line
 	4150 2600 4150 2550
+$Comp
+L VUSB #PWR?
+U 1 1 59873DF1
+P 2100 3050
+F 0 "#PWR?" H 2100 2900 50  0001 C CNN
+F 1 "VUSB" H 2100 3200 50  0000 C CNN
+F 2 "" H 2100 3050 50  0001 C CNN
+F 3 "" H 2100 3050 50  0001 C CNN
+	1    2100 3050
+	1    0    0    -1
+$EndComp
+$Comp
+L VUSB #PWR?
+U 1 1 59874131
+P 1800 4500
+F 0 "#PWR?" H 1800 4350 50  0001 C CNN
+F 1 "VUSB" H 1800 4650 50  0000 C CNN
+F 2 "" H 1800 4500 50  0001 C CNN
+F 3 "" H 1800 4500 50  0001 C CNN
+	1    1800 4500
+	1    0    0    -1
+$EndComp
+Wire Wire Line
+	1900 4700 1800 4700
+Wire Wire Line
+	1800 4700 1800 4500
+$Comp
+L VUSB #PWR?
+U 1 1 598741DF
+P 4200 4100
+F 0 "#PWR?" H 4200 3950 50  0001 C CNN
+F 1 "VUSB" H 4200 4250 50  0000 C CNN
+F 2 "" H 4200 4100 50  0001 C CNN
+F 3 "" H 4200 4100 50  0001 C CNN
+	1    4200 4100
+	0    -1   -1   0
+$EndComp
+$Comp
+L VUSB #PWR?
+U 1 1 598745B3
+P 5450 4850
+F 0 "#PWR?" H 5450 4700 50  0001 C CNN
+F 1 "VUSB" H 5450 5000 50  0000 C CNN
+F 2 "" H 5450 4850 50  0001 C CNN
+F 3 "" H 5450 4850 50  0001 C CNN
+	1    5450 4850
+	-1   0    0    1
+$EndComp
+Wire Wire Line
+	5950 4700 5950 4900
+Wire Wire Line
+	6050 4700 6050 4900
+Wire Wire Line
+	6650 4100 7000 4100
+Text GLabel 7000 4100 2    60   Output ~ 0
+USB_CHR0
+Text GLabel 5950 4900 3    60   Output ~ 0
+USB_CHREN
+Text GLabel 6050 4900 3    60   Output ~ 0
+USB_CHR1
 $EndSCHEMATC
